File: C128Diag.kicad_sch (KiCad schematic)
At the start: 60 parts, among them J1 CP1, J2 CP2, J3 KB, J4 Cas, J5 Vid, J6 Serial, J7 UP, P1 1k, U1 4066, U10 74LS04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

Commit message: Fixed potentiometer footprint.
Parts:
- P1: footprint Potentiometer_THT:Potentiometer_Bourns_3339P_Vertical -> C128Diag:Potentiometer_Bourns_3339P_Vertical
Changed lines of the file:
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@@
   (title_block
     (title "C128Diag")
-    (date "2023-05-04")
-    (rev "0")
+    (date "2023-05-16")
+    (rev "1")
     (company "www.hackup.net")
     (comment 1 "Creative Commons Attribution-NonCommercial-ShareAlike 4.0 International License.")
@@
       (effects (font (size 1.27 1.27)) (justify right))
     )
-    (property "Footprint" "Potentiometer_THT:Potentiometer_Bourns_3339P_Vertical" (at 87.63 227.33 0)
+    (property "Footprint" "C128Diag:Potentiometer_Bourns_3339P_Vertical" (at 87.63 227.33 0)
       (effects (font (size 1.27 1.27)) hide)
     )

Commit message: Adding connector wiring to schematics.
Parts:
- J5: value Vid -> Aud
Connections:
- net SER1: now reaches J6.1 (Pin_1), U10.1, U10.5, U11.1, U7.1, U7.13
- net KB6: now reaches J3.9 (Pin_9), U3.1 (X1)
- net KB20: now reaches J3.7 (Pin_7), U3.10 (X4)
- net KB3: now reaches J3.11 (Pin_11), U3.11 (Y4)
- net KB23: now reaches J3.4 (Pin_4), U3.2 (Y1)
- net KB21: now reaches J3.6 (Pin_6), U3.3 (X2)
- net KB4: now reaches J3.10 (Pin_10), U3.4 (Y2)
- net KB2: now reaches J3.12 (Pin_12), U3.8 (X3)
- net KB1: now reaches J3.13 (Pin_13), U3.9 (Y3)
- net SER5: now reaches J6.2 (Pin_2), U10.3, U11.9, U7.10, U8.13
- net CP1_6: now reaches J1.1 (Pin_1), U1.1 (X1)
- net CP2_3: now reaches J2.3 (Pin_3), U1.10 (X4)
- net CP1_3: now reaches J1.3 (Pin_3), U1.11 (Y4)
- net CP2_6: now reaches J2.1 (Pin_1), U1.2 (Y1)
- net CP2_4: now reaches J2.2 (Pin_2), U1.3 (X2)
- net CP1_4: now reaches J1.2 (Pin_2), U1.4 (Y2)
- net CP1_2: now reaches J1.4 (Pin_4), U1.8 (X3)
- net CP2_2: now reaches J2.4 (Pin_4), U1.9 (Y3)
- net KB16: now reaches J3.3 (Pin_3), U5.16 (B2)
- net KB17: now reaches J3.2 (Pin_2), U5.17 (B1)
- net KB18: now reaches J3.1 (Pin_1), U5.18 (B0)
- net KB22: now reaches J3.5 (Pin_5), U2.10 (X4)
- net KB9: now reaches J3.8 (Pin_8), U2.11 (Y4)
- net CP2_1: now reaches J2.5 (Pin_5), U2.3 (X2)
- net CP1_1: now reaches J1.5 (Pin_5), U2.4 (Y2)
- net AV5: now reaches J5.1 (Pin_1), U2.1 (X1)
Other:
- added sheet C128Diag Connectors (C128Diag-Connectors.kicad_sch)
- moved on the sheet: C2, C3, J1, J2, J3, J4, J5, J6, J7, JU1, JU2, JU3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
