File: C128Diag-Connectors.kicad_sch (KiCad schematic)
At the start: 10 parts, among them J10 CP2, J11 IEC, J12 A/V, J13 A/V, J8 Keyboard, J9 CP1

Commit message: Added missing user port connector wiring, fixes #1.
Parts:
- added D1, D2: LED, symbol Device:LED_Small
- added J14: C64-UserPort, Hackup_Commodore:C64-User-Port-Female, symbol hackup-commodore:C64-UserPort
- added R10: 680R, symbol Device:R_Small
- added R9: 330R, symbol Device:R_Small
Connections:
- new net: D1.1 (K), R9.2
- new net: D1.2 (A), J14.2 (5V)
- new net: D2.1 (K), R10.2
- new net: D2.2 (A), J14.11 (9VAC2)
- new net: J14.1 (GND2), R9.1
- new net: J14.10 (9VAC1), R10.1
- new net: J14.8 (/PC2), J14.B (/FLAG2)
- new net: J14.9 (ATN), J14.M (PA2)
- new net: J14.C (PB0), J14.H (PB4)
- new net: J14.D (PB1), J14.J (PB5)
- new net: J14.E (PB2), J14.K (PB6)
- new net: J14.F (PB3), J14.L (PB7)
- new net UP6: J14.6 (CNT2)
- new net UP7: J14.7 (SP2)
- no-connect marks 10 -> 16
